File: tinker_kad/Fantabulous Inari-Kieran.brd (EAGLE design)
At the start: 68.6 x 53.3 mm, 13 parts

Commit message: tinkercad project add
Parts:
- added PIEZO1: (no value), AUTODESK_CIRCUITS_BREADBOARD:PIEZO-22MM
Connections:
- removed net N$10 (its old number): SB_AZUL.2, SB_AZUL.4, U1.5
- removed net N$8 (its old number): R2.1, R3.1, R4.1, R5.1, SB_AMARELO.1, SB_AMARELO.3, SB_AZUL.1, SB_AZUL.3, SB_BRANCO.1, SB_BRANCO.3, SB_LARANJA.1, SB_LARANJA.3, U1.GND.
- removed net N$9 (its old number): SB_LARANJA.2, SB_LARANJA.4, U1.4
- new net N$13: SB_AZUL.2, SB_AZUL.4, U1.6
- new net N$14: PIEZO1.P$2, R2.1, R3.1, R4.1, R5.1, SB_AMARELO.1, SB_AMARELO.3, SB_AZUL.1, SB_AZUL.3, SB_BRANCO.1, SB_BRANCO.3, SB_LARANJA.1, SB_LARANJA.3, U1.GND.
- new net N$15: PIEZO1.P$1, U1.7
- new net N$5: SB_BRANCO.2, SB_BRANCO.4, U1.3
- net N$6: now also SB_AMARELO.2, SB_AMARELO.4, U1.4; no longer SB_BRANCO.2, SB_BRANCO.4, U1.2
- net N$7: now also SB_LARANJA.2, SB_LARANJA.4, U1.5; no longer SB_AMARELO.2, SB_AMARELO.4, U1.3

Commit message: projeto atualizado tinker-kad
Parts:
- renumbered DL_AMARELO to DL_Yellow, DL_LARANJA to DL_Orange, SB_BRANCO to SB_Yellow
Connections:
- new net N$16: SB_AMARELO.2
- new net N$17: SB_AMARELO.1
- new net N$18: SB_AMARELO.3, U1.6
- new net N$19: DL_AZUL.A, U1.9
- new net N$20: DL_Yellow.A, U1.8
- new net N$21: DL_BRANCO.A, U1.11
- new net N$4: DL_Yellow.K, R2.2
- net N$1: now also SB_Yellow.2; no longer DL_AZUL.K, R2.2
- net N$11: now also PIEZO1.P$2, R2.1, R3.1, R4.1, R5.1, SB_AMARELO.4, SB_AZUL.4, SB_LARANJA.4, SB_Yellow.4, U1.GND..; no longer DL_AZUL.A, U1.11
- net N$12: now also SB_LARANJA.2; no longer U1.5V
- net N$13: now also SB_LARANJA.1; no longer SB_AZUL.2, SB_AZUL.4, U1.6
- net N$14: now also U1.5; no longer PIEZO1.P$2, R2.1, R3.1, R4.1, R5.1, SB_AMARELO.1, SB_AMARELO.3, SB_AZUL.1, SB_AZUL.3, SB_LARANJA.1, SB_Yellow.1, SB_Yellow.3, U1.GND.
- net N$2: now also SB_Yellow.1; no longer DL_Orange.K, R3.2
- net N$3: now also SB_Yellow.3, U1.3; no longer DL_Yellow.K, R4.2
- net N$5: now also DL_AZUL.K, R3.2; no longer SB_Yellow.2, SB_Yellow.4, U1.3
- net N$6: now also SB_AZUL.2; no longer SB_AMARELO.2, SB_AMARELO.4, U1.4
- net N$7: now also SB_AZUL.1; no longer SB_LARANJA.2, SB_LARANJA.4, U1.5
- net N$8: now also SB_AZUL.3, U1.4; no longer DL_BRANCO.A, U1.8
- net N$9: now also DL_Orange.K, R4.2; no longer DL_Yellow.A, U1.9
